File: atx2/atx2.sch (KiCad schematic (older format))
At the start: 6 parts, among them J1 ATX-24, J2 Conn_02x02_Top_Bottom, J3 Conn_01x02, J4 Conn_01x02, J5 Conn_01x02, J6 Conn_02x02_Top_Bottom

Commit message: design-v1
Parts:
- removed J2, J6: Conn_02x02_Top_Bottom, Connector_TE-Connectivity:TE_MATE-N-LOK_1-770874-x_2x02_P4.14mm_Vertical, symbol Connector_Generic:Conn_02x02_Top_Bottom
- added D1, D2, D3, D4, D5, D6: LED, LED_SMD:LED_1206_3216Metric, symbol Device:LED
- added J2: Conn_02x04_Top_Bottom, Connector_Molex:Molex_Mini-Fit_Jr_5566-08A2_2x04_P4.20mm_Vertical, symbol Connector_Generic:Conn_02x04_Top_Bottom
- added J7, J8, J9: Conn_01x02, TerminalBlock:TerminalBlock_Wuerth_691311400102_P7.62mm, symbol Connector_Generic:Conn_01x02
- added R1, R4, R5: 220, Resistor_SMD:R_1206_3216Metric, symbol Device:R
- added R2, R3: 510, Resistor_SMD:R_1206_3216Metric, symbol Device:R
- added R6: 68, Resistor_SMD:R_1206_3216Metric, symbol Device:R
- added SW1: SW_SPDT, Button_Switch_THT:SW_E-Switch_EG1271_DPDT, symbol Switch:SW_SPDT
- J1: footprint Connector_TE-Connectivity:TE_MATE-N-LOK_1-794072-x_2x12_P4.14mm_Vertical -> Connector_Molex:Molex_Mini-Fit_Jr_5566-24A2_2x12_P4.20mm_Vertical
Connections:
- net +12V: now also J2.5 (Pin_5), J2.6 (Pin_6), J2.7 (Pin_7), J2.8 (Pin_8), R2.2
- net +5V: now also R5.2
- net GND: now also D1.1 (K), D2.1 (K), D4.1 (K), D5.1 (K), D6.1 (K), J2.1 (Pin_1), J2.2 (Pin_2), J2.3 (Pin_3), J2.4 (Pin_4), J7.2 (Pin_2), J8.2 (Pin_2), J9.2 (Pin_2), R3.2, SW1.1 (A); no longer J1.16 (PS_ON#)
- net +3V3: now reaches J1.1 (+3.3V), J1.12 (+3.3V), J1.13 (+3.3V), J1.2 (+3.3V)
- net +3V3: now also J7.1 (Pin_1), R6.2
- net -12V: now reaches J1.14 (-12V)
- net -12V: now also D3.1 (K), J9.1 (Pin_1)
- net at J1.8 (PWR_OK): now also R1.2
- net +5VA: now reaches J1.9 (+5VSB)
- net +5VA: now also J8.1 (Pin_1), R4.2
- new net: J1.16 (PS_ON#), SW1.2 (B)
- new net: D1.2 (A), R1.1
- new net: D2.2 (A), R2.1
- new net: D3.2 (A), R3.1
- new net: D4.2 (A), R4.1
- new net: D5.2 (A), R5.1
- new net: D6.2 (A), R6.1
- no-connect marks 4 -> 0
